Commit message: entendido launch file y hecho que el coche se vea y mueva en gazebo

File: src/car_controller/urdf/car.ros2_control.xacro (robot description, xacro)
@@ -22,8 +22,8 @@
             </joint>
         </xacro:macro>
-        <xacro:rueda nombre="base_rueda_trasera_izquierda"/>
-        <xacro:rueda nombre="base_rueda_trasera_derecha"/>
-        <xacro:rueda nombre="base_rueda_delantera_izquierda"/>
-        <xacro:rueda nombre="base_rueda_delantera_derecha"/>
+        <xacro:rueda nombre="rueda_trasera_izquierda_joint"/>
+        <xacro:rueda nombre="rueda_trasera_derecha_joint"/>
+        <xacro:rueda nombre="rueda_delantera_izquierda_joint"/>
+        <xacro:rueda nombre="rueda_delantera_derecha_joint"/>
     </ros2_control>
 </robot>

File: src/car_controller/urdf/car.urdf.xacro (robot description, xacro)
@@ -22,5 +22,5 @@
                 <mesh filename="package://car_controller/meshes/chasis.stl" scale="0.0016 0.0016 0.0016"/>
             </geometry>
-            <origin xyz="0.0 0.0 0.0" rpy="0.0 0.0 0.0"/>
+            <origin xyz="0.0 0.0 0.0" rpy="0.0 0.0 ${pi/2}"/>
             <material name="red"/>
         </visual>
@@ -53,15 +53,15 @@
             <xacro:inercia_inicial mass="0.1"></xacro:inercia_inicial>
         </link>
-        <joint name="base_rueda_${nombre}" type="continuous">
+        <joint name="rueda_${nombre}_joint" type="continuous">
             <parent link="base"/>
             <child link="rueda_${nombre}"/>
-            <origin xyz="${dx} ${dy} -0.038" rpy="0.0 ${pi/2} 0.0"/>
-            <axis xyz="0.0 0.0 1.0"/>
+            <origin xyz="${dx} ${dy} -0.038" rpy="${pi/2} 0.0 0.0"/>
+            <axis xyz="0.0 0.0 -1.0"/>
         </joint>
     </xacro:macro>
-    <xacro:rueda nombre="trasera_izquierda" dx="0.065" dy="0.106" />
-    <xacro:rueda nombre="trasera_derecha" dx="-0.065" dy="0.106" />
-    <xacro:rueda nombre="delantera_izquierda" dx="0.065" dy="-0.116" />
-    <xacro:rueda nombre="delantera_derecha" dx="-0.065" dy="-0.116" />
+    <xacro:rueda nombre="trasera_izquierda" dx="0.116" dy="0.065"/>
+    <xacro:rueda nombre="trasera_derecha" dx="0.116" dy="-0.065"/>
+    <xacro:rueda nombre="delantera_izquierda" dx="-0.106" dy="0.065" />
+    <xacro:rueda nombre="delantera_derecha" dx="-0.106" dy="-0.065" />
     <xacro:include filename="$(find car_controller)/urdf/car.ros2_control.xacro"/>
     <xacro:include filename="$(find car_controller)/urdf/car.gazebo.xacro"/>
